Commit message: Running Test

File: p3dx_description/urdf/pioneer3dx_wheel.xacro (robot description, xacro)
@@ -87,7 +87,11 @@
     <transmission name="${parent}_${suffix}_wheel_trans">
       <type>pr2_mechanism_model/SimpleTransmission</type>
-      <joint name="base_${suffix}_wheel_joint" />
+      <joint name="base_${suffix}_wheel_joint">
+      	<hardwareInterface>EffortJointInterface</hardwareInterface>
+      	<!-- <hardwareInterface>VelocityJointInterface</hardwareInterface> -->
+      </joint>
       <actuator name="base_${suffix}_wheel_motor">
         <hardwareInterface>EffortJointInterface</hardwareInterface>
+        <!-- <hardwareInterface>VelocityJointInterface</hardwareInterface> -->
         <mechanicalReduction>${reflect * 624/35 * 80/19}</mechanicalReduction>
       </actuator>
