Commit message: camera plugin added

File: p3dx_description/urdf/p3dx.urdf (robot description, URDF)
Before this commit: robot pioneer3dx, 13 links, 12 joints
Links:
- added link world
Joints:
- joint camera_plate_joint: origin xyz=2 2 1.0 rpy=0 0 0 -> xyz=1 1 0.0 rpy=0 0 0; parent base_link -> world

File: p3dx_description/urdf/pioneer3dx.xacro (robot description, xacro)
@@ -223,3 +223,58 @@
 		<child link="lms100" />
 	</joint>
+	<xacro:property name="camera_length" value="0.05"/>
+	<xacro:property name="camera_plate_radius" value="0.1"/>
+	<xacro:property name="camera_plate_length" value="0.02"/>
+	<!-- camera joint -->
+	<link name="camera_plate">
+		<collision>
+			<origin xyz="0 0 ${camera_plate_length/2}" rpy="0 0 0"/>
+			<geometry>
+				<cylinder radius="${camera_plate_radius}" length="${camera_plate_length}"/>
+			</geometry>
+		</collision>
+		<visual>
+			<origin xyz="0 0 ${camera_plate_length/2}" rpy="0 0 0"/>
+			<geometry>
+				<cylinder radius="${camera_plate_radius}" length="${camera_plate_length}"/>
+			</geometry>
+			<material name="white"/>
+		</visual>
+		<!-- TODO: inertial should be added-->
+		<inertial>
+			<mass value="0.1"/>
+			<origin xyz="0 0 0" rpy="0 0 0"/>
+			<inertia ixx="0.1" ixy="0" ixz="0" iyy="0.1" iyz="0" izz="0.1" />
+		</inertial>
+	</link>
+	<joint name="camera_plate_joint" type="fixed">
+		<origin xyz="0.1 0 0.01" rpy="0 0 0"/>
+		<parent link="top_plate"/>
+		<child link="camera_plate"/>
+	</joint>
+	<link name="front_camera_link">
+		<collision>
+			<origin xyz="0 0 ${camera_length/2}" rpy="0 0 0"/>
+			<geometry>
+				<box size="${camera_length} ${camera_length} ${camera_length}"/>
+			</geometry>
+		</collision>
+		<visual>
+			<origin xyz="0 0 ${camera_length/2}" rpy="0 0 0"/>
+			<geometry>
+				<box size="${camera_length} ${camera_length} ${camera_length}"/>
+			</geometry>
+			<material name="black"/>
+		</visual>
+		<inertial>
+			<mass value="1e-5"/>
+			<origin xyz="0 0 ${-1*camera_length/2}" rpy="0 0 0"/>
+			<inertia ixx="1e-6" ixy="0" ixz="0" iyy="1e-6" iyz="0" izz="1e-6" />
+		</inertial>
+	</link>
+	<joint name="front_camera_joint" type="fixed">
+		<origin xyz="${camera_plate_radius - camera_length/2} 0 ${camera_plate_length}" rpy="0 0 0"/>
+		<parent link="camera_plate"/>
+		<child link="front_camera_link"/>
+	</joint>
 </robot>
